Commit message: modify the missing motors

File: hexapod_urdf_2/urdf/hexapod_urdf_2.urdf (robot description, URDF)
Before this commit: robot hexapod_complete_urdf, 19 links, 18 joints
Links:
- link body: mass 0.163675340720187 -> 0.38148; geometry collision mesh filename=package://hexapod_urdf_2/meshes/body.STL; visual mesh filename=package://hexapod_urdf_2/meshes/body.STL
- link calf1: mass 0.0333887237767673 -> 0.0696897389529788; geometry collision mesh filename=package://hexapod_urdf_2/meshes/calf1.STL; visual mesh filename=package://hexapod_urdf_2/meshes/calf1.STL
- link calf2: mass 0.0333887237767673 -> 0.0696897389529788; geometry collision mesh filename=package://hexapod_urdf_2/meshes/calf2.STL; visual mesh filename=package://hexapod_urdf_2/meshes/calf2.STL
- link calf3: mass 0.0333887237767673 -> 0.0696897389529788; geometry collision mesh filename=package://hexapod_urdf_2/meshes/calf3.STL; visual mesh filename=package://hexapod_urdf_2/meshes/calf3.STL
- link calf4: mass 0.0333887237767673 -> 0.06969; geometry collision mesh filename=package://hexapod_urdf_2/meshes/calf4.STL; visual mesh filename=package://hexapod_urdf_2/meshes/calf4.STL
- link calf5: mass 0.0333887237767673 -> 0.06969; geometry collision mesh filename=package://hexapod_urdf_2/meshes/calf5.STL; visual mesh filename=package://hexapod_urdf_2/meshes/calf5.STL
- link calf6: mass 0.0333887237767674 -> 0.06969; geometry collision mesh filename=package://hexapod_urdf_2/meshes/calf6.STL; visual mesh filename=package://hexapod_urdf_2/meshes/calf6.STL
- link haunch1: mass 0.0165574984042957 -> 0.0528585135805074; geometry collision mesh filename=package://hexapod_urdf_2/meshes/haunch1.STL; visual mesh filename=package://hexapod_urdf_2/meshes/haunch1.STL
- link haunch2: mass 0.0165574984042958 -> 0.0528585135805073; geometry collision mesh filename=package://hexapod_urdf_2/meshes/haunch2.STL; visual mesh filename=package://hexapod_urdf_2/meshes/haunch2.STL
- link haunch3: mass 0.0165574984042957 -> 0.0528585135805073; geometry collision mesh filename=package://hexapod_urdf_2/meshes/haunch3.STL; visual mesh filename=package://hexapod_urdf_2/meshes/haunch3.STL
- link haunch4: mass 0.0165574984042958 -> 0.0528585135805073; geometry collision mesh filename=package://hexapod_urdf_2/meshes/haunch4.STL; visual mesh filename=package://hexapod_urdf_2/meshes/haunch4.STL
- link haunch5: mass 0.0165574984042957 -> 0.0528585135805073; geometry collision mesh filename=package://hexapod_urdf_2/meshes/haunch5.STL; visual mesh filename=package://hexapod_urdf_2/meshes/haunch5.STL
- link haunch6: mass 0.0165574984042958 -> 0.052859; geometry collision mesh filename=package://hexapod_urdf_2/meshes/haunch6.STL; visual mesh filename=package://hexapod_urdf_2/meshes/haunch6.STL
- link thigh1: mass 0.0266777976712455 -> 0.026678; geometry collision mesh filename=package://hexapod_urdf_2/meshes/thigh1.STL; visual mesh filename=package://hexapod_urdf_2/meshes/thigh1.STL
- link thigh2: geometry collision mesh filename=package://hexapod_urdf_2/meshes/thigh2.STL; visual mesh filename=package://hexapod_urdf_2/meshes/thigh2.STL
- link thigh3: geometry collision mesh filename=package://hexapod_urdf_2/meshes/thigh3.STL; visual mesh filename=package://hexapod_urdf_2/meshes/thigh3.STL
- link thigh4: geometry collision mesh filename=package://hexapod_urdf_2/meshes/thigh4.STL; visual mesh filename=package://hexapod_urdf_2/meshes/thigh4.STL
- link thigh5: geometry collision mesh filename=package://hexapod_urdf_2/meshes/thigh5.STL; visual mesh filename=package://hexapod_urdf_2/meshes/thigh5.STL
- link thigh6: geometry collision mesh filename=package://hexapod_urdf_2/meshes/thigh6.STL; visual mesh filename=package://hexapod_urdf_2/meshes/thigh6.STL
Joints:
- joint jo_calf1: axis 0.6065 -0.79508 0 -> 0.488032087614086 -0.872825687900532 0; origin xyz=-0.059467 -0.045362 -0.051836 rpy=0 0 0 -> xyz=-0.0794271375992236 -0.0444109199730361 0 rpy=0 0 0
- joint jo_calf2: axis 0.97865 0.20554 0 -> 0.99905921046351 -0.0433669688591199 0; origin xyz=0.016375 -0.077966 -0.043979 rpy=0 0 0 -> xyz=-0.00345491629745502 -0.0795920498747716 -0.0439791899666504 rpy=0 0 0
- joint jo_calf3: axis -0.57082 0.82108 0 -> -0.570818413422048 0.821076329520183 0; origin xyz=0.062191 0.043236 -0.050438 rpy=0 0 0 -> xyz=0.0621910510159125 0.043235684422541 -0.050437572959575 rpy=0 0 0
- joint jo_calf4: axis 0.42566 0.90488 0 -> 0.425663753099527 0.904881411731518 0; origin xyz=0.064518 -0.03035 -0.056545 rpy=0 0 0 -> xyz=0.064517858471575 -0.0303497380130774 -0.0565450204773114 rpy=0 0 0
- joint jo_calf5: origin xyz=-0.00655141272371919 0.0778994038600545 -0.0465807027595338 rpy=0 0 0 -> xyz=-0.00655141272371994 0.0778994038600507 -0.0465807027595325 rpy=0 0 0
- joint jo_haunch4: origin xyz=0.055591 -0.055049 -0.0088 rpy=0 0 -0.20877 -> xyz=0.0555906522089202 -0.0550491214110074 -0.00880000000000555 rpy=0 0 -0.208770544653029
- joint jo_haunch6: origin xyz=-0.0555906522088054 0.0550491214109962 -0.00880000000000014 rpy=0 0 -0.208770544653029 -> xyz=-0.055591 0.055049 -0.0088 rpy=0 0 -0.20877
- joint jo_thigh1: axis 0.6065 -0.79508 0 -> 0.488032087614086 -0.872825687900532 0; origin xyz=-0.030819 -0.027282 0.01015 rpy=0 0 0 -> xyz=-0.0343653982253839 -0.0226521942604925 0.0101500000000387 rpy=0 0 0
- joint jo_thigh2: axis 0.97865 0.20554 0 -> 0.99906 -0.043367 0; origin xyz=0.011374 -0.039557 0.01015 rpy=0 0 0 -> xyz=0.001217 -0.041141 0.01015 rpy=0 0 0
- joint jo_thigh3: origin xyz=0.0319927280865342 0.0258953248595354 0.0101500000000014 rpy=0 0 0 -> xyz=0.0319927280865405 0.0258953248595306 0.0101499999999997 rpy=0 0 0
- joint jo_thigh5: axis -0.99648 -0.083805 0 -> -0.996482166521584 -0.0838050822113381 0; origin xyz=-0.0064296 0.040654 0.01015 rpy=0 0 0 -> xyz=-0.0064296451243417 0.0406541776890781 0.01015 rpy=0 0 0
- joint jo_thigh6: axis -0.42566 -0.90488 0 -> -0.425663753099532 -0.904881411731515 0; origin xyz=-0.038422 0.014759 0.01015 rpy=0 0 0 -> xyz=-0.0384223732108755 0.0147588528295395 0.0101499999999933 rpy=0 0 0

File: mujoco_hexapod_2/hexapod_urdf_2.urdf (robot description, URDF)
Before this commit: robot hexapod_complete_urdf, 19 links, 18 joints
Links:
- link body: mass 0.163675340720187 -> 0.38148; geometry collision mesh filename=meshes/body.STL; visual mesh filename=meshes/body.STL
- link calf1: mass 0.0333887237767673 -> 0.0696897389529788; geometry collision mesh filename=meshes/calf1.STL; visual mesh filename=meshes/calf1.STL
- link calf2: mass 0.0333887237767673 -> 0.0696897389529788; geometry collision mesh filename=meshes/calf2.STL; visual mesh filename=meshes/calf2.STL
- link calf3: mass 0.0333887237767673 -> 0.0696897389529788; geometry collision mesh filename=meshes/calf3.STL; visual mesh filename=meshes/calf3.STL
- link calf4: mass 0.0333887237767673 -> 0.06969; geometry collision mesh filename=meshes/calf4.STL; visual mesh filename=meshes/calf4.STL
- link calf5: mass 0.0333887237767673 -> 0.06969; geometry collision mesh filename=meshes/calf5.STL; visual mesh filename=meshes/calf5.STL
- link calf6: mass 0.0333887237767674 -> 0.06969; geometry collision mesh filename=meshes/calf6.STL; visual mesh filename=meshes/calf6.STL
- link haunch1: mass 0.0165574984042957 -> 0.0528585135805074; geometry collision mesh filename=meshes/haunch1.STL; visual mesh filename=meshes/haunch1.STL
- link haunch2: mass 0.0165574984042958 -> 0.0528585135805073; geometry collision mesh filename=meshes/haunch2.STL; visual mesh filename=meshes/haunch2.STL
- link haunch3: mass 0.0165574984042957 -> 0.0528585135805073; geometry collision mesh filename=meshes/haunch3.STL; visual mesh filename=meshes/haunch3.STL
- link haunch4: mass 0.0165574984042958 -> 0.0528585135805073; geometry collision mesh filename=meshes/haunch4.STL; visual mesh filename=meshes/haunch4.STL
- link haunch5: mass 0.0165574984042957 -> 0.0528585135805073; geometry collision mesh filename=meshes/haunch5.STL; visual mesh filename=meshes/haunch5.STL
- link haunch6: mass 0.0165574984042958 -> 0.052859; geometry collision mesh filename=meshes/haunch6.STL; visual mesh filename=meshes/haunch6.STL
- link thigh1: mass 0.0266777976712455 -> 0.026678; geometry collision mesh filename=meshes/thigh1.STL; visual mesh filename=meshes/thigh1.STL
- link thigh2: geometry collision mesh filename=meshes/thigh2.STL; visual mesh filename=meshes/thigh2.STL
- link thigh3: geometry collision mesh filename=meshes/thigh3.STL; visual mesh filename=meshes/thigh3.STL
- link thigh4: geometry collision mesh filename=meshes/thigh4.STL; visual mesh filename=meshes/thigh4.STL
- link thigh5: geometry collision mesh filename=meshes/thigh5.STL; visual mesh filename=meshes/thigh5.STL
- link thigh6: geometry collision mesh filename=meshes/thigh6.STL; visual mesh filename=meshes/thigh6.STL
Joints:
- joint jo_calf1: axis 0.6065 -0.79508 0 -> 0.488032087614086 -0.872825687900532 0; origin xyz=-0.059467 -0.045362 -0.051836 rpy=0 0 0 -> xyz=-0.0794271375992236 -0.0444109199730361 0 rpy=0 0 0
- joint jo_calf2: axis 0.97865 0.20554 0 -> 0.99905921046351 -0.0433669688591199 0; origin xyz=0.016375 -0.077966 -0.043979 rpy=0 0 0 -> xyz=-0.00345491629745502 -0.0795920498747716 -0.0439791899666504 rpy=0 0 0
- joint jo_calf3: axis -0.57082 0.82108 0 -> -0.570818413422048 0.821076329520183 0; origin xyz=0.062191 0.043236 -0.050438 rpy=0 0 0 -> xyz=0.0621910510159125 0.043235684422541 -0.050437572959575 rpy=0 0 0
- joint jo_calf4: axis 0.42566 0.90488 0 -> 0.425663753099527 0.904881411731518 0; origin xyz=0.064518 -0.03035 -0.056545 rpy=0 0 0 -> xyz=0.064517858471575 -0.0303497380130774 -0.0565450204773114 rpy=0 0 0
- joint jo_calf5: origin xyz=-0.00655141272371919 0.0778994038600545 -0.0465807027595338 rpy=0 0 0 -> xyz=-0.00655141272371994 0.0778994038600507 -0.0465807027595325 rpy=0 0 0
- joint jo_haunch4: origin xyz=0.055591 -0.055049 -0.0088 rpy=0 0 -0.20877 -> xyz=0.0555906522089202 -0.0550491214110074 -0.00880000000000555 rpy=0 0 -0.208770544653029
- joint jo_haunch6: origin xyz=-0.0555906522088054 0.0550491214109962 -0.00880000000000014 rpy=0 0 -0.208770544653029 -> xyz=-0.055591 0.055049 -0.0088 rpy=0 0 -0.20877
- joint jo_thigh1: axis 0.6065 -0.79508 0 -> 0.488032087614086 -0.872825687900532 0; origin xyz=-0.030819 -0.027282 0.01015 rpy=0 0 0 -> xyz=-0.0343653982253839 -0.0226521942604925 0.0101500000000387 rpy=0 0 0
- joint jo_thigh2: axis 0.97865 0.20554 0 -> 0.99906 -0.043367 0; origin xyz=0.011374 -0.039557 0.01015 rpy=0 0 0 -> xyz=0.001217 -0.041141 0.01015 rpy=0 0 0
- joint jo_thigh3: origin xyz=0.0319927280865342 0.0258953248595354 0.0101500000000014 rpy=0 0 0 -> xyz=0.0319927280865405 0.0258953248595306 0.0101499999999997 rpy=0 0 0
- joint jo_thigh5: axis -0.99648 -0.083805 0 -> -0.996482166521584 -0.0838050822113381 0; origin xyz=-0.0064296 0.040654 0.01015 rpy=0 0 0 -> xyz=-0.0064296451243417 0.0406541776890781 0.01015 rpy=0 0 0
- joint jo_thigh6: axis -0.42566 -0.90488 0 -> -0.425663753099532 -0.904881411731515 0; origin xyz=-0.038422 0.014759 0.01015 rpy=0 0 0 -> xyz=-0.0384223732108755 0.0147588528295395 0.0101499999999933 rpy=0 0 0
